Commit message: ajuste das chamas

File: p_g5_description/urdf/p_g5.gazebo.xacro (robot description, xacro)
@@ -168,3 +168,7 @@
     </sensor>
   </gazebo>
+  <gazebo reference="flame_right_link">
+<!--    <material>Gazebo/DarkGrey</material>-->
+    <material>Gazebo/Orange</material>
+  </gazebo>
 </robot>

File: p_g5_description/urdf/p_g5.urdf.xacro (robot description, xacro)
@@ -189,20 +189,19 @@
   <link name="camera_rgb_optical_frame"/>
 <!--  acresentar chamas laterais -->
+  <link name="flame_right_link">
+    <visual>
+      <origin xyz="0 0 0" rpy="0 0 0"/>
+      <geometry>
+        <mesh filename="package://p_g5_description/mesh/flaming_gear_keychain.stl" scale="0.004 0.004 0.01"/>
+<!--        <mesh filename="package://turtlebot3_description/meshes/sensors/lds.stl" scale="0.001 0.001 0.001"/>-->
+<!--        <cylinder length="0.018" radius="0.033"/>-->
+      </geometry>
+    </visual>
+  </link>
   <joint name="base_link_to_flame_rigth_link" type="fixed">
-    <parent link="base_link"/>
-    <child link="flame_rigth_link"/>
-    <origin xyz="1.0 1 1.023" rpy="2 0 0"/>
-  </joint>
-  <link name="flame_right_link">
-    <visual>
-      <origin xyz="0 0 0" rpy="1.57 0 0"/>
-      <geometry>
-<!--        <mesh filename="package://p_g5_description/mesh/flaming_gear_keychain.stl" scale="0.001 0.001 0.001"/>-->
-<!--        <mesh filename="package://turtlebot3_description/meshes/sensors/lds.stl" scale="0.001 0.001 0.001"/>-->
-        <cylinder length="0.018" radius="0.033"/>
-      </geometry>
-      <material name="dark"/>
-<!--      <material name="orange"/>-->
-    </visual>
-  </link>
+    <origin xyz="0 0 0.3" rpy="0 0 0"/>
+    <parent link="base_link"/>
+    <child link="flame_right_link"/>
+    <material name="orange"/>
+  </joint>
 </robot>

Commit message: finalizacao da chama left

File: p_g5_description/urdf/p_g5.gazebo.xacro (robot description, xacro)
@@ -168,5 +168,5 @@
     </sensor>
   </gazebo>
-  <gazebo reference="flame_right_link">
+  <gazebo reference="flame_left_link">
 <!--    <material>Gazebo/DarkGrey</material>-->
     <material>Gazebo/Orange</material>

File: p_g5_description/urdf/p_g5.urdf.xacro (robot description, xacro)
@@ -189,9 +189,9 @@
   <link name="camera_rgb_optical_frame"/>
 <!--  acresentar chamas laterais -->
-  <link name="flame_right_link">
-    <visual>
-      <origin xyz="0 0 0" rpy="0 0 0"/>
-      <geometry>
-        <mesh filename="package://p_g5_description/mesh/flaming_gear_keychain.stl" scale="0.004 0.004 0.01"/>
+  <link name="flame_left_link">
+    <visual>
+      <origin xyz="0 0 0" rpy="0 1.57 1.57"/>
+      <geometry>
+        <mesh filename="package://p_g5_description/mesh/flaming_gear_keychain.stl" scale="0.002 0.0035 0.005"/>
 <!--        <mesh filename="package://turtlebot3_description/meshes/sensors/lds.stl" scale="0.001 0.001 0.001"/>-->
 <!--        <cylinder length="0.018" radius="0.033"/>-->
@@ -199,8 +199,8 @@
     </visual>
   </link>
-  <joint name="base_link_to_flame_rigth_link" type="fixed">
-    <origin xyz="0 0 0.3" rpy="0 0 0"/>
-    <parent link="base_link"/>
-    <child link="flame_right_link"/>
+  <joint name="base_link_to_flame_left_link" type="fixed">
+    <origin xyz="-0.169 0.12 0.05" rpy="0 0 0"/>
+    <parent link="base_link"/>
+    <child link="flame_left_link"/>
     <material name="orange"/>
   </joint>

Commit message: finalizacao das 2 chamas

File: p_g5_description/urdf/p_g5.gazebo.xacro (robot description, xacro)
@@ -168,7 +168,12 @@
     </sensor>
   </gazebo>
+<!--color in flame-->
   <gazebo reference="flame_left_link">
 <!--    <material>Gazebo/DarkGrey</material>-->
     <material>Gazebo/Orange</material>
   </gazebo>
+    <gazebo reference="flame_right_link">
+<!--    <material>Gazebo/DarkGrey</material>-->
+    <material>Gazebo/Orange</material>
+  </gazebo>
 </robot>

File: p_g5_description/urdf/p_g5.urdf.xacro (robot description, xacro)
@@ -189,4 +189,5 @@
   <link name="camera_rgb_optical_frame"/>
 <!--  acresentar chamas laterais -->
+<!--  chama esquerda-->
   <link name="flame_left_link">
     <visual>
@@ -205,3 +206,20 @@
     <material name="orange"/>
   </joint>
+<!--  chama direita-->
+  <link name="flame_right_link">
+    <visual>
+      <origin xyz="0 0 0" rpy="0 -1.57 1.57"/>
+      <geometry>
+        <mesh filename="package://p_g5_description/mesh/flaming_gear_keychain.stl" scale="0.002 0.0035 0.005"/>
+<!--        <mesh filename="package://turtlebot3_description/meshes/sensors/lds.stl" scale="0.001 0.001 0.001"/>-->
+<!--        <cylinder length="0.018" radius="0.033"/>-->
+      </geometry>
+    </visual>
+  </link>
+  <joint name="base_link_to_flame_right_link" type="fixed">
+    <origin xyz="-0.169 -0.12 0.05" rpy="0 0 0"/>
+    <parent link="base_link"/>
+    <child link="flame_right_link"/>
+    <material name="orange"/>
+  </joint>
 </robot>

Commit message: finalixacao do xacro.launch

File: p_g5_description/urdf/p_g5.gazebo.xacro (robot description, xacro)
@@ -5,6 +5,6 @@
   <xacro:arg name="imu_visual"    default="false"/>
   <gazebo reference="base_link">
-<!--    <material>Gazebo/DarkGrey</material>-->
-    <material>Gazebo/Orange</material>
+    <material>Gazebo/DarkGrey</material>
+<!--    <material>Gazebo/Orange</material>-->
   </gazebo>
   <gazebo reference="wheel_left_link">
@@ -16,5 +16,6 @@
     <maxVel>0.1</maxVel>
     <fdir1>1 0 0</fdir1>
-    <material>Gazebo/FlatBlack</material>
+<!--    <material>Gazebo/FlatBlack</material>-->
+    <material>Gazebo/Orange</material>
   </gazebo>
   <gazebo reference="wheel_right_link">
@@ -26,5 +27,6 @@
     <maxVel>0.1</maxVel>
     <fdir1>1 0 0</fdir1>
-    <material>Gazebo/FlatBlack</material>
+<!--    <material>Gazebo/FlatBlack</material>-->
+    <material>Gazebo/Orange</material>
   </gazebo>
   <gazebo reference="caster_back_right_link">

File: p_g5_description/urdf/p_g5.urdf.xacro (robot description, xacro)
@@ -15,6 +15,6 @@
         <mesh filename="package://turtlebot3_description/meshes/bases/waffle_pi_base.stl" scale="0.001 0.001 0.001"/>
       </geometry>
-<!--      <material name="light_black"/>-->
-      <material name="orange"/>
+      <material name="light_black"/>
+<!--      <material name="orange"/>-->
     </visual>
     <collision>
@@ -44,6 +44,6 @@
         <mesh filename="package://turtlebot3_description/meshes/wheels/left_tire.stl" scale="0.001 0.001 0.001"/>
       </geometry>
-      <material name="dark"/>
-<!--      <material name="orange"/>-->
+<!--      <material name="dark"/>-->
+      <material name="orange"/>
     </visual>
     <collision>
@@ -73,6 +73,6 @@
         <mesh filename="package://turtlebot3_description/meshes/wheels/right_tire.stl" scale="0.001 0.001 0.001"/>
       </geometry>
-      <material name="dark"/>
-<!--      <material name="orange"/>-->
+<!--      <material name="dark"/>-->
+      <material name="orange"/>
     </visual>
     <collision>
