Commit message: Finalização do Read me Correção do common_properties.xacro Inclusão do package fnr para o novo world

File: p_g5_description/urdf/common_properties.xacro (robot description, xacro)
@@ -2,5 +2,5 @@
 <robot name="xacro_properties" xmlns:xacro="http://ros.org/wiki/xacro">
   <!-- Init colour -->
-  <material name="black">
+  <material name="Black">
       <color rgba="0.0 0.0 0.0 1.0"/>
   </material>
@@ -11,5 +11,5 @@
     <color rgba="0.05 0.05 0.05 1.0"/>
   </material>
-  <material name="light_black">
+  <material name="LightBlack">
     <color rgba="0.4 0.4 0.4 1.0"/>
   </material>
@@ -26,15 +26,9 @@
     <color rgba="${255/255} ${108/255} ${10/255} 1.0"/>
   </material>
-  <material name="brown">
+  <material name="Brown">
     <color rgba="${222/255} ${207/255} ${195/255} 1.0"/>
-  </material>
-  <material name="red">
-    <color rgba="0.8 0.0 0.0 1.0"/>
   </material>
     <material name="Red">
     <color rgba="0.8 0.0 0.0 1.0"/>
-  </material>
-  <material name="white">
-    <color rgba="1.0 1.0 1.0 1.0"/>
   </material>
     <material name="White">
