Commit message: Criação do launch file spawn Nome do jogador e cores como argumentos de entrada no launch file spawn Utilizacão do controlador ros_diff_drive.gazebo.xacro Criacao do teleop.launch Configuracao do Rviz

File: p_g5_description/urdf/p_g5.gazebo.macro.xacro (robot description, xacro)
@@ -1,9 +1,10 @@
 <?xml version="1.0"?>
-<robot name="turtlebot3_waffle_pi_sim" xmlns:xacro="http://ros.org/wiki/xacro">
+<robot name="p_g5_gaz" xmlns:xacro="http://ros.org/wiki/xacro">
+  <xacro:include filename="$(find p_g5_description)/urdf/ros_diff_drive.gazebo.xacro"/>
   <xacro:arg name="laser_visual"  default="false"/>
   <xacro:arg name="camera_visual" default="false"/>
   <xacro:arg name="imu_visual"    default="false"/>
   <gazebo reference="base_link">
-    <material>Gazebo/DarkGrey</material>
+    <material>Gazebo/${base_color}</material>
   </gazebo>
   <gazebo reference="wheel_left_link">
@@ -15,5 +16,5 @@
     <maxVel>0.1</maxVel>
     <fdir1>1 0 0</fdir1>
-    <material>Gazebo/Orange</material>
+    <material>Gazebo/${player_color}</material>
   </gazebo>
   <gazebo reference="wheel_right_link">
@@ -25,6 +26,5 @@
     <maxVel>0.1</maxVel>
     <fdir1>1 0 0</fdir1>
-<!--    <material>Gazebo/FlatBlack</material>-->
-    <material>Gazebo/Orange</material>
+   <material>Gazebo/${player_color}</material>
   </gazebo>
   <gazebo reference="caster_back_right_link">
@@ -53,5 +53,5 @@
     <material>Gazebo/Grey</material>
   </gazebo>
-  <gazebo>
+  <!--<gazebo>
     <plugin name="turtlebot3_waffle_pi_controller" filename="libgazebo_ros_diff_drive.so">
       <commandTopic>cmd_vel</commandTopic>
@@ -74,5 +74,5 @@
       <rosDebugLevel>na</rosDebugLevel>
     </plugin>
-  </gazebo>
+  </gazebo>-->
   <gazebo>
     <plugin name="imu_plugin" filename="libgazebo_ros_imu.so">
@@ -104,5 +104,5 @@
   </gazebo>
   <gazebo reference="base_scan">
-    <material>Gazebo/FlatBlack</material>
+    <material>Gazebo/${scan_color}</material>
     <sensor type="ray" name="lds_lfcd_sensor">
       <pose>0 0 0 0 0 0</pose>
@@ -171,9 +171,9 @@
   <gazebo reference="flame_left_link">
 <!--    <material>Gazebo/DarkGrey</material>-->
-    <material>Gazebo/Orange</material>
+    <material>Gazebo/${player_color}</material>
   </gazebo>
     <gazebo reference="flame_right_link">
 <!--    <material>Gazebo/DarkGrey</material>-->
-    <material>Gazebo/Orange</material>
+    <material>Gazebo/${player_color}</material>
   </gazebo>
 </robot>

File: p_g5_description/urdf/p_g5.urdf.xacro (robot description, xacro)
@@ -1,6 +1,10 @@
 <?xml version="1.0" ?>
-<robot name="turtlebot3_waffle_pi" xmlns:xacro="http://ros.org/wiki/xacro">
-  <xacro:include filename="$(find turtlebot3_description)/urdf/common_properties.xacro"/>
-  <xacro:include filename="$(find p_g5_description)/urdf/p_g5.gazebo.xacro"/>
+<robot name="$(arg player_name)" xmlns:xacro="http://ros.org/wiki/xacro">
+  <xacro:include filename="$(find p_g5_description)/urdf/common_properties.xacro"/>
+  <xacro:property name="player_name" value="$(arg player_name)"/>
+  <xacro:property name="player_color" value="$(arg player_color)"/>
+  <xacro:property name="base_color" value="$(arg base_color)"/>
+  <xacro:property name="scan_color" value="$(arg scan_color)"/>
+  <xacro:include filename="$(find p_g5_description)/urdf/p_g5.gazebo.macro.xacro"/>
   <link name="base_footprint"/>
   <joint name="base_joint" type="fixed">
@@ -15,6 +19,5 @@
         <mesh filename="package://turtlebot3_description/meshes/bases/waffle_pi_base.stl" scale="0.001 0.001 0.001"/>
       </geometry>
-      <material name="light_black"/>
-<!--      <material name="orange"/>-->
+      <material name="${base_color}"/>
     </visual>
     <collision>
@@ -44,6 +47,5 @@
         <mesh filename="package://turtlebot3_description/meshes/wheels/left_tire.stl" scale="0.001 0.001 0.001"/>
       </geometry>
-<!--      <material name="dark"/>-->
-      <material name="orange"/>
+      <material name="${player_color}"/>
     </visual>
     <collision>
@@ -74,5 +76,5 @@
       </geometry>
 <!--      <material name="dark"/>-->
-      <material name="orange"/>
+      <material name="${player_color}"/>
     </visual>
     <collision>
@@ -147,5 +149,5 @@
         <mesh filename="package://turtlebot3_description/meshes/sensors/lds.stl" scale="0.001 0.001 0.001"/>
       </geometry>
-      <material name="dark"/>
+      <material name="${scan_color}"/>
     </visual>
     <collision>
@@ -195,7 +197,6 @@
       <geometry>
         <mesh filename="package://p_g5_description/mesh/flaming_gear_keychain.stl" scale="0.002 0.0035 0.005"/>
-<!--        <mesh filename="package://turtlebot3_description/meshes/sensors/lds.stl" scale="0.001 0.001 0.001"/>-->
-<!--        <cylinder length="0.018" radius="0.033"/>-->
-      </geometry>
+      </geometry>
+      <material name="${player_color}"/>
     </visual>
   </link>
@@ -204,5 +205,4 @@
     <parent link="base_link"/>
     <child link="flame_left_link"/>
-    <material name="orange"/>
   </joint>
 <!--  chama direita-->
@@ -212,7 +212,6 @@
       <geometry>
         <mesh filename="package://p_g5_description/mesh/flaming_gear_keychain.stl" scale="0.002 0.0035 0.005"/>
-<!--        <mesh filename="package://turtlebot3_description/meshes/sensors/lds.stl" scale="0.001 0.001 0.001"/>-->
-<!--        <cylinder length="0.018" radius="0.033"/>-->
-      </geometry>
+      </geometry>
+      <material name="${player_color}"/>
     </visual>
   </link>
@@ -221,5 +220,4 @@
     <parent link="base_link"/>
     <child link="flame_right_link"/>
-    <material name="orange"/>
   </joint>
 </robot>

Commit message: alteracoes reuniao

File: p_g5_description/urdf/p_g5.gazebo.macro.xacro (robot description, xacro)
@@ -105,5 +105,5 @@
   </gazebo>
   <gazebo reference="base_scan">
-    <material>Gazebo/${scan_color}</material>
+    <material>Gazebo/${player_color}</material>
     <sensor type="ray" name="lds_lfcd_sensor">
       <pose>0 0 0 0 0 0</pose>
@@ -144,6 +144,8 @@
           <horizontal_fov>1.085595</horizontal_fov>
           <image>
-              <width>640</width>
-              <height>480</height>
+<!--              <width>640</width>-->
+<!--              <height>480</height>-->
+             <width>1680</width>
+              <height>1050</height>
               <format>R8G8B8</format>
           </image>

File: p_g5_description/urdf/p_g5.urdf.xacro (robot description, xacro)
@@ -149,5 +149,5 @@
         <mesh filename="package://turtlebot3_description/meshes/sensors/lds.stl" scale="0.001 0.001 0.001"/>
       </geometry>
-      <material name="${scan_color}"/>
+      <material name="${player_color}"/>
     </visual>
     <collision>

Commit message: contacts and Gmapping

File: p_g5_description/urdf/p_g5.gazebo.macro.xacro (robot description, xacro)
@@ -180,3 +180,17 @@
     <material>Gazebo/${player_color}</material>
   </gazebo>
+<!--  Bumper sensor-->
+<gazebo reference="base_link">
+    <sensor name="base_link" type="contact">
+      <update_rate>1000.0</update_rate>
+      <always_on>true</always_on>
+      <contact>
+        <collision>base_footprint_fixed_joint_lump__base_link_collision</collision>
+      </contact>
+      <plugin name="base_link_contact_sensor_plugin" filename="libgazebo_ros_bumper.so">
+        <bumperTopicName>contact</bumperTopicName>
+        <frameName>${player_color}/world</frameName>
+      </plugin>
+    </sensor>
+  </gazebo>
 </robot>

File: p_g5_description/urdf/p_g5.urdf.xacro (robot description, xacro)
@@ -1,9 +1,14 @@
 <?xml version="1.0" ?>
 <robot name="$(arg player_name)" xmlns:xacro="http://ros.org/wiki/xacro">
+<!--<robot name="p_g5" xmlns:xacro="http://ros.org/wiki/xacro">-->
   <xacro:include filename="$(find p_g5_description)/urdf/common_properties.xacro"/>
-  <xacro:property name="player_name" value="$(arg player_name)"/>
-  <xacro:property name="player_color" value="$(arg player_color)"/>
-  <xacro:property name="base_color" value="$(arg base_color)"/>
-  <xacro:property name="scan_color" value="$(arg scan_color)"/>
+  <xacro:property name="player_name" value="$(arg player_name)"  />
+  <xacro:property name="player_color" value="$(arg player_color)"  />
+  <xacro:property name="base_color" value="$(arg base_color)" />
+  <xacro:property name="scan_color" value="$(arg scan_color)" />
+<!--  <xacro:property name="player_name" default="p_g5" />-->
+<!--  <xacro:property name="player_color" default="Orange" />-->
+<!--  <xacro:property name="base_color" default="DarkGrey"/>-->
+<!--  <xacro:property name="scan_color" default="FlatBlack"/>-->
   <xacro:include filename="$(find p_g5_description)/urdf/p_g5.gazebo.macro.xacro"/>
   <link name="base_footprint"/>
