Commit message: colocar a flames laterais

File: p_g5_description/urdf/p_g5.urdf.xacro (robot description, xacro)
@@ -189,18 +189,20 @@
   <link name="camera_rgb_optical_frame"/>
 <!--  acresentar chamas laterais -->
-<!--  <link name="flame_right_link">-->
-<!--    <visual>-->
-<!--      <origin xyz="0 0 0" rpy="1.57 0 0"/>-->
-<!--      <geometry>-->
+  <joint name="base_link_to_flame_rigth_link" type="fixed">
+    <parent link="base_link"/>
+    <child link="flame_rigth_link"/>
+    <origin xyz="1.0 1 1.023" rpy="2 0 0"/>
+  </joint>
+  <link name="flame_right_link">
+    <visual>
+      <origin xyz="0 0 0" rpy="1.57 0 0"/>
+      <geometry>
 <!--        <mesh filename="package://p_g5_description/mesh/flaming_gear_keychain.stl" scale="0.001 0.001 0.001"/>-->
-<!--      </geometry>-->
-<!--      <material name="dark"/>-->
-<!--&lt;!&ndash;      <material name="orange"/>&ndash;&gt;-->
-<!--    </visual>-->
-<!--  </link>-->
-<!--   <joint name="base_link_to_flame_rigth_link" type="fixed">-->
-<!--    <parent link="base_link"/>-->
-<!--    <child link="flame_rigth_link"/>-->
-<!--    <origin xyz="0.0 0.144 0.023" rpy="-1.57 0 0"/>-->
-<!--  </joint>-->
+<!--        <mesh filename="package://turtlebot3_description/meshes/sensors/lds.stl" scale="0.001 0.001 0.001"/>-->
+        <cylinder length="0.018" radius="0.033"/>
+      </geometry>
+      <material name="dark"/>
+<!--      <material name="orange"/>-->
+    </visual>
+  </link>
 </robot>

Commit message: finalizacao das 2 chamas pequena correcoes

File: p_g5_description/urdf/p_g5.urdf.xacro (robot description, xacro)
@@ -218,5 +218,5 @@
   </link>
   <joint name="base_link_to_flame_right_link" type="fixed">
-    <origin xyz="-0.169 -0.12 0.05" rpy="0 0 0"/>
+    <origin xyz="-0.169 -0.12 0.044" rpy="0 0 0"/>
     <parent link="base_link"/>
     <child link="flame_right_link"/>

Commit message: Orientações corretas

File: p_g5_description/urdf/p_g5.urdf.xacro (robot description, xacro)
@@ -7,4 +7,5 @@
   <xacro:property name="base_color" value="$(arg base_color)" />
   <xacro:property name="scan_color" value="$(arg scan_color)" />
+   <xacro:property name="orientacao" value="$(arg orientacao)" />
 <!--  <xacro:property name="player_name" default="p_g5" />-->
 <!--  <xacro:property name="player_color" default="Orange" />-->
@@ -16,5 +17,5 @@
     <parent link="base_footprint"/>
     <child link="base_link" />
-    <origin xyz="0 0 0.010" rpy="0 0 0"/>
+    <origin xyz="0 0 0.010" rpy="0 0 ${orientacao}"/>
   </joint>
   <link name="base_link">
